Commit message: Adding axis_direction support to the CyberGear hardware interface.
The mecanum_drive_controller ignores the URDF joint axes, so mirror-mounted wheels need the sign flip in the hardware plugin. The optional axis_direction parameter (1 or -1, default 1) is applied to the feedback in read() and to the commands in write().

File: cybergear_ros2_control/cybergear_control/description/ros2_control/cybergear.ros2_control.urdf.xacro (robot description, xacro)
@@ -1,5 +1,5 @@
 <?xml version="1.0"?>
 <robot xmlns:xacro="http://www.ros.org/wiki/xacro">
-  <xacro:macro name="cybergear_ros2_control" params="name canbus motor_type device_id kp kd joint_name">
+  <xacro:macro name="cybergear_ros2_control" params="name canbus motor_type device_id kp kd joint_name axis_direction:=1">
     <ros2_control name="${name}" type="actuator">
         <hardware>
@@ -14,4 +14,5 @@
             <param name="kd">${kd}</param>
             <param name="calibrate_on_activate">false</param>
+            <param name="axis_direction">${axis_direction}</param>
         </hardware>
         <joint name="${joint_name}">
